File: battery_capacity.kicad_pcb (KiCad board)
At the start: 2 copper layers, 47 x 48 mm, 17 parts, among them J1 Screw_Terminal_01x03, J2 Screw_Terminal_01x04, Q1 IRLML2060, Q2 IRLML2060, U1 PC817, U2 PC817, U3 YAAJ_DCDC_StepDown_LM2596

Commit message: h
Parts:
- moved U3 2.54 mm to (144.8, 101.6)
Routing:
- net +24V: track 82.8 -> 81.4 mm
Other:
- board size 47 x 48 mm -> 47 x 45 mm
