File: battery_capacity.kicad_sch (KiCad schematic)
At the start: 17 parts, among them J1 Screw_Terminal_01x03, J2 Screw_Terminal_01x04, Q1 IRLML2060, Q2 IRLML2060, U1 PC817, U2 PC817, U3 YAAJ_DCDC_StepDown_LM2596

Commit message: h
Parts:
- removed J1: Screw_Terminal_01x03, TerminalBlock_Altech:Altech_AK300_1x03_P5.00mm_45-Degree, symbol Connector:Screw_Terminal_01x03
- added J3: Screw_Terminal_01x04, TerminalBlock_Altech:Altech_AK300_1x04_P5.00mm_45-Degree, symbol Connector:Screw_Terminal_01x04
Connections:
- net GND: now also J3.3 (Pin_3)
- net at R4.1: now also J3.1 (Pin_1)
- net at R5.1: now also J3.2 (Pin_2)
- net +5V: now reaches U3.4 (Vout)
- net +5V: now also J3.4 (Pin_4)
Changed lines of the file:
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@@
+    (stroke (width 0) (type default))
+  )
+  (wire (pts (xy 62.23 86.36) (xy 64.77 86.36))
     (stroke (width 0) (type default))
   )
@@
     (stroke (width 0) (type default))
   )
-  (wire (pts (xy 71.12 83.82) (xy 64.77 83.82))
+  (wire (pts (xy 62.23 83.82) (xy 71.12 83.82))
     (stroke (width 0) (type default))
   )
@@
     (stroke (width 0) (type default))
   )
-  (wire (pts (xy 64.77 81.28) (xy 74.93 81.28))
+  (wire (pts (xy 62.23 81.28) (xy 74.93 81.28))
     (stroke (width 0) (type default))
   )
@@
     )
   )
+  (symbol (lib_id "power:+5V") (at 62.23 88.9 180) (unit 1)
+    (in_bom yes) (on_board yes) (dnp no) (fields_autoplaced)
+    (property "Reference" "#PWR013" (at 62.23 85.09 0)
+      (effects (font (size 1.27 1.27)) hide)
+    )
+    (property "Value" "+5V" (at 62.23 93.98 0)
+      (effects (font (size 1.27 1.27)))
+    )
+    (property "Footprint" "" (at 62.23 88.9 0)
+      (effects (font (size 1.27 1.27)) hide)
+    )
+    (property "Datasheet" "" (at 62.23 88.9 0)
+      (effects (font (size 1.27 1.27)) hide)
+    )
+    (pin "1")
+    (instances
+      (project "battery_capacity"
+        (path "/dc426f08-c2a9-4db5-a4cb-5d963ec2c2f2"
+          (reference "#PWR013") (unit 1)
+        )
+      )
+    )
+  )
   (symbol (lib_id "Transistor_FET:IRLML2060") (at 133.35 121.92 0) (unit 1)
     (in_bom yes) (on_board yes) (dnp no) (fields_autoplaced)
@@
     )
   )
+  (symbol (lib_id "Connector:Screw_Terminal_01x04") (at 57.15 83.82 0) (mirror y) (unit 1)
+    (in_bom yes) (on_board yes) (dnp no)
+    (property "Reference" "J3" (at 54.61 84.455 0)
+      (effects (font (size 1.27 1.27)) (justify left))
+    )
+    (property "Value" "Screw_Terminal_01x04" (at 54.61 86.995 0)
+      (effects (font (size 1.27 1.27)) (justify left))
+    )
+    (property "Footprint" "TerminalBlock_Altech:Altech_AK300_1x04_P5.00mm_45-Degree" (at 57.15 83.82 0)
+      (effects (font (size 1.27 1.27)) hide)
+    )
+    (property "Datasheet" "~" (at 57.15 83.82 0)
+      (effects (font (size 1.27 1.27)) hide)
+    )
+    (pin "1")
+    (pin "2")
+    (pin "3")
+    (pin "4")
+    (instances
+      (project "battery_capacity"
+        (path "/dc426f08-c2a9-4db5-a4cb-5d963ec2c2f2"
+          (reference "J3") (unit 1)
+        )
+      )
+    )
+  )
   (symbol (lib_id "power:GND") (at 135.89 97.79 0) (unit 1)
     (in_bom yes) (on_board yes) (dnp no) (fields_autoplaced)
@@
     )
   )
+  (symbol (lib_id "power:+5V") (at 118.11 156.21 180) (unit 1)
+    (in_bom yes) (on_board yes) (dnp no) (fields_autoplaced)
+    (property "Reference" "#PWR014" (at 118.11 152.4 0)
+      (effects (font (size 1.27 1.27)) hide)
+    )
+    (property "Value" "+5V" (at 118.11 161.29 0)
+      (effects (font (size 1.27 1.27)))
+    )
+    (property "Footprint" "" (at 118.11 156.21 0)
+      (effects (font (size 1.27 1.27)) hide)
+    )
+    (property "Datasheet" "" (at 118.11 156.21 0)
+      (effects (font (size 1.27 1.27)) hide)
+    )
+    (pin "1")
+    (instances
+      (project "battery_capacity"
+        (path "/dc426f08-c2a9-4db5-a4cb-5d963ec2c2f2"
+          (reference "#PWR014") (unit 1)
+        )
+      )
+    )
+  )
   (symbol (lib_id "Device:R") (at 78.74 81.28 90) (unit 1)
     (in_bom yes) (on_board yes) (dnp no) (fields_autoplaced)
@@
         )
       )
-    )
-  )
-  (symbol (lib_id "Connector:Screw_Terminal_01x03") (at 59.69 83.82 0) (mirror y) (unit 1)
-    (in_bom yes) (on_board yes) (dnp no)
-    (property "Reference" "J1" (at 59.69 91.44 0)
-      (effects (font (size 1.27 1.27)))
-    )
-    (property "Value" "Screw_Terminal_01x03" (at 59.69 88.9 0)
-      (effects (font (size 1.27 1.27)))
-    )
-    (property "Footprint" "TerminalBlock_Altech:Altech_AK300_1x03_P5.00mm_45-Degree" (at 59.69 83.82 0)
-      (effects (font (size 1.27 1.27)) hide)
-    )
-    (property "Datasheet" "~" (at 59.69 83.82 0)
-      (effects (font (size 1.27 1.27)) hide)
-    )
-    (pin "1")
-    (pin "2")
-    (pin "3")
-    (instances
-      (project "battery_capacity"
-        (path "/dc426f08-c2a9-4db5-a4cb-5d963ec2c2f2"
-          (reference "J1") (unit 1)
-        )
-      )
